File: hardware/mica.kicad_pcb (KiCad board)
At the start: 0 parts

Commit message: Remove 4 of the 8 mounting holes
Parts:
- added C1: 100n, Capacitor_SMD:C_0402_1005Metric, F.Cu at (60.2, 78.3)
- added C10: 1u, Capacitor_SMD:C_0402_1005Metric, F.Cu at (71.7, 97.6)
- added C11: 47n, Capacitor_SMD:C_0402_1005Metric, F.Cu at (74.6, 97.6)
- added C12: 47n, Capacitor_SMD:C_0402_1005Metric, F.Cu at (71.7, 99.6)
- added C13: 10n, Capacitor_SMD:C_0402_1005Metric, F.Cu at (74.6, 99.6)
- added C14: 2.2u, Capacitor_SMD:C_0402_1005Metric, F.Cu at (77.5, 95.6)
- added C15: 100n, Capacitor_SMD:C_0402_1005Metric, F.Cu at (74.6, 95.6)
- added C16: 100n, Capacitor_SMD:C_0402_1005Metric, F.Cu at (55.9, 112.7)
- added C17: 1u, Capacitor_SMD:C_0402_1005Metric, F.Cu at (51.4, 116.7)
- added C18: 47n, Capacitor_SMD:C_0402_1005Metric, F.Cu at (54.3, 116.7)
- added C19: 47n, Capacitor_SMD:C_0402_1005Metric, F.Cu at (51.4, 118.7)
- added C2: 100n, Capacitor_SMD:C_0402_1005Metric, F.Cu at (46.5, 94.2)
- added C20: 10n, Capacitor_SMD:C_0402_1005Metric, F.Cu at (54.2, 118.6)
- added C21: 2.2u, Capacitor_SMD:C_0402_1005Metric, F.Cu at (57.2, 114.7)
- added C22: 100n, Capacitor_SMD:C_0402_1005Metric, F.Cu at (54.3, 114.7)
- added C23: 100n, Capacitor_SMD:C_0402_1005Metric, F.Cu at (38.4, 112.7)
- added C24: 1u, Capacitor_SMD:C_0402_1005Metric, F.Cu at (33.9, 116.7)
- added C25: 47n, Capacitor_SMD:C_0402_1005Metric, F.Cu at (36.8, 116.7)
- added C26: 47n, Capacitor_SMD:C_0402_1005Metric, F.Cu at (33.9, 118.7)
- added C27: 10n, Capacitor_SMD:C_0402_1005Metric, F.Cu at (36.8, 118.6)
- added C28: 2.2u, Capacitor_SMD:C_0402_1005Metric, F.Cu at (39.7, 114.7)
- added C29: 100n, Capacitor_SMD:C_0402_1005Metric, F.Cu at (36.8, 114.7)
- added C3: 100n, Capacitor_SMD:C_0402_1005Metric, F.Cu at (38.5, 102.8)
- added C30: 100n, Capacitor_SMD:C_0402_1005Metric, F.Cu at (76.2, 80.3)
- added C31: 1u, Capacitor_SMD:C_0402_1005Metric, F.Cu at (71.7, 84.3)
- added C32: 47n, Capacitor_SMD:C_0402_1005Metric, F.Cu at (74.6, 84.2)
- added C33: 47n, Capacitor_SMD:C_0402_1005Metric, F.Cu at (71.7, 86.2)
- added C34: 10n, Capacitor_SMD:C_0402_1005Metric, F.Cu at (74.6, 86.2)
- added C35: 2.2u, Capacitor_SMD:C_0402_1005Metric, F.Cu at (77.5, 82.3)
- added C36: 100n, Capacitor_SMD:C_0402_1005Metric, F.Cu at (74.6, 82.3)
- added C37: 100n, Capacitor_SMD:C_0402_1005Metric, F.Cu at (93.7, 80.3)
- added C38: 1u, Capacitor_SMD:C_0402_1005Metric, F.Cu at (89.2, 84.3)
- added C39: 47n, Capacitor_SMD:C_0402_1005Metric, F.Cu at (92.1, 84.2)
- added C4: 100n, Capacitor_SMD:C_0402_1005Metric, F.Cu at (51.2, 86.2)
- added C40: 47n, Capacitor_SMD:C_0402_1005Metric, F.Cu at (89.2, 86.2)
- added C41: 10n, Capacitor_SMD:C_0402_1005Metric, F.Cu at (92.1, 86.2)
- added C42: 2.2u, Capacitor_SMD:C_0402_1005Metric, F.Cu at (95.0, 82.3)
- added C43: 100n, Capacitor_SMD:C_0402_1005Metric, F.Cu at (92.1, 82.3)
- added C44: 100n, Capacitor_SMD:C_0402_1005Metric, F.Cu at (93.7, 93.6)
- added C45: 1u, Capacitor_SMD:C_0402_1005Metric, F.Cu at (89.2, 97.6)
- added C46: 47n, Capacitor_SMD:C_0402_1005Metric, F.Cu at (92.1, 97.6)
- added C47: 47n, Capacitor_SMD:C_0402_1005Metric, F.Cu at (89.2, 99.6)
- added C48: 10n, Capacitor_SMD:C_0402_1005Metric, F.Cu at (92.1, 99.6)
- added C49: 2.2u, Capacitor_SMD:C_0402_1005Metric, F.Cu at (95.0, 95.6)
- added C5: 100n, Capacitor_SMD:C_0402_1005Metric, F.Cu at (57.4, 80.3)
- added C50: 100n, Capacitor_SMD:C_0402_1005Metric, F.Cu at (92.1, 95.6)
- added C51: 100n, Capacitor_SMD:C_0402_1005Metric, F.Cu at (21.0, 112.7)
- added C52: 1u, Capacitor_SMD:C_0402_1005Metric, F.Cu at (16.4, 116.7)
- added C53: 47n, Capacitor_SMD:C_0402_1005Metric, F.Cu at (19.4, 116.7)
- added C54: 47n, Capacitor_SMD:C_0402_1005Metric, F.Cu at (16.4, 118.7)
- added C55: 10n, Capacitor_SMD:C_0402_1005Metric, F.Cu at (19.3, 118.6)
- added C56: 2.2u, Capacitor_SMD:C_0402_1005Metric, F.Cu at (22.2, 114.7)
- added C57: 100n, Capacitor_SMD:C_0402_1005Metric, F.Cu at (19.4, 114.7)
- added C58: 100n, Capacitor_SMD:C_0402_1005Metric, F.Cu at (76.2, 107.0)
- added C59: 1u, Capacitor_SMD:C_0402_1005Metric, F.Cu at (71.7, 111.0)
- added C6: 2.2u, Capacitor_SMD:C_0402_1005Metric, F.Cu at (48.3, 88.2)
- added C60: 47n, Capacitor_SMD:C_0402_1005Metric, F.Cu at (74.6, 111.0)
- added C61: 47n, Capacitor_SMD:C_0402_1005Metric, F.Cu at (71.7, 112.9)
- added C62: 10n, Capacitor_SMD:C_0402_1005Metric, F.Cu at (74.6, 112.9)
- added C63: 2.2u, Capacitor_SMD:C_0402_1005Metric, F.Cu at (77.5, 109.0)
- added C64: 100n, Capacitor_SMD:C_0402_1005Metric, F.Cu at (74.6, 109.0)
- added C7: 470p, Capacitor_SMD:C_0402_1005Metric, F.Cu at (57.4, 78.3)
- added C8: 2.2u, Capacitor_SMD:C_0402_1005Metric, F.Cu at (31.9, 103.8)
- added C9: 100n, Capacitor_SMD:C_0402_1005Metric, F.Cu at (76.2, 93.6)
- added D1: LED_Red, LED_SMD:LED_0603_1608Metric, F.Cu at (22.7, 104.1)
- added D2: LED_Green, LED_SMD:LED_0603_1608Metric, F.Cu at (11.9, 103.7)
- added F1: Polyfuse_Small, Fuse:Fuse_1206_3216Metric, F.Cu at (12.7, 100.8)
- added H1: MountingHole, MountingHole:MountingHole_3.2mm_M3, F.Cu at (105.5, 56.6)
- added H2: MountingHole, MountingHole:MountingHole_3.2mm_M3, F.Cu at (105.8, 144.7)
- added H3: MountingHole, MountingHole:MountingHole_3.2mm_M3, F.Cu at (195.1, 144.5)
- added H4: MountingHole, MountingHole:MountingHole_3.2mm_M3, F.Cu at (194.2, 54.6)
- added J1: USB_C_Receptacle_USB2.0, User:USB_C_Receptacle_HRO_TYPE-C-31-M-12, F.Cu at (15.7, 83.1)
- added J2: Conn_ARM_JTAG_SWD_10, User:Samtec_FTSH-105-01-L-DV-K, F.Cu at (26.4, 90.3)
- added MK1: AP3722AT, User:AllPower_AP3722AT_3.76x2.24mm, F.Cu at (67.1, 93.3)
- added MK2: AP3722AT, User:AllPower_AP3722AT_3.76x2.24mm, F.Cu at (46.7, 112.4)
- added MK3: AP3722AT, User:AllPower_AP3722AT_3.76x2.24mm, F.Cu at (29.2, 112.4)
- added MK4: AP3722AT, User:AllPower_AP3722AT_3.76x2.24mm, F.Cu at (67.1, 80.0)
- added MK5: AP3722AT, User:AllPower_AP3722AT_3.76x2.24mm, F.Cu at (84.5, 80.0)
- added MK6: AP3722AT, User:AllPower_AP3722AT_3.76x2.24mm, F.Cu at (84.5, 93.3)
- added MK7: AP3722AT, User:AllPower_AP3722AT_3.76x2.24mm, F.Cu at (11.8, 112.4)
- added MK8: AP3722AT, User:AllPower_AP3722AT_3.76x2.24mm, F.Cu at (67.1, 106.7)
- added R1: 10k, Resistor_SMD:R_0402_1005Metric, F.Cu at (26.1, 103.8)
- added R10: 1k, Resistor_SMD:R_0402_1005Metric, F.Cu at (70.5, 91.7)
- added R11: 499k, Resistor_SMD:R_0402_1005Metric, F.Cu at (73.4, 93.7)
- added R12: 1M, Resistor_SMD:R_0402_1005Metric, F.Cu at (50.1, 112.7)
- added R13: 1M, Resistor_SMD:R_0402_1005Metric, F.Cu at (55.9, 110.7)
- added R14: 1M, Resistor_SMD:R_0402_1005Metric, F.Cu at (51.4, 114.7)
- added R15: 1Meg, Resistor_SMD:R_0402_1005Metric, F.Cu at (53.0, 110.7)
- added R16: 1k, Resistor_SMD:R_0402_1005Metric, F.Cu at (50.1, 110.7)
- added R17: 499k, Resistor_SMD:R_0402_1005Metric, F.Cu at (53.0, 112.7)
- added R18: 1M, Resistor_SMD:R_0402_1005Metric, F.Cu at (32.6, 112.7)
- added R19: 1M, Resistor_SMD:R_0402_1005Metric, F.Cu at (38.5, 110.7)
- added R2: 5.1k, Resistor_SMD:R_0402_1005Metric, F.Cu at (15.4, 104.6)
- added R20: 1M, Resistor_SMD:R_0402_1005Metric, F.Cu at (33.9, 114.7)
- added R21: 1Meg, Resistor_SMD:R_0402_1005Metric, F.Cu at (35.5, 110.7)
- added R22: 1k, Resistor_SMD:R_0402_1005Metric, F.Cu at (32.6, 110.7)
- added R23: 499k, Resistor_SMD:R_0402_1005Metric, F.Cu at (35.5, 112.7)
- added R24: 1M, Resistor_SMD:R_0402_1005Metric, F.Cu at (70.5, 80.3)
- added R25: 1M, Resistor_SMD:R_0402_1005Metric, F.Cu at (76.3, 78.3)
- added R26: 1M, Resistor_SMD:R_0402_1005Metric, F.Cu at (71.8, 82.3)
- added R27: 1Meg, Resistor_SMD:R_0402_1005Metric, F.Cu at (73.4, 78.3)
- added R28: 1k, Resistor_SMD:R_0402_1005Metric, F.Cu at (70.5, 78.3)
- added R29: 499k, Resistor_SMD:R_0402_1005Metric, F.Cu at (73.4, 80.3)
- added R3: 5.1k, Resistor_SMD:R_0402_1005Metric, F.Cu at (48.4, 86.3)
- added R30: 1M, Resistor_SMD:R_0402_1005Metric, F.Cu at (87.9, 80.3)
- added R31: 1M, Resistor_SMD:R_0402_1005Metric, F.Cu at (93.7, 78.3)
- added R32: 1M, Resistor_SMD:R_0402_1005Metric, F.Cu at (89.2, 82.3)
- added R33: 1Meg, Resistor_SMD:R_0402_1005Metric, F.Cu at (90.8, 78.3)
- added R34: 1k, Resistor_SMD:R_0402_1005Metric, F.Cu at (87.9, 78.3)
- added R35: 499k, Resistor_SMD:R_0402_1005Metric, F.Cu at (90.8, 80.3)
- added R36: 1M, Resistor_SMD:R_0402_1005Metric, F.Cu at (87.9, 93.7)
- added R37: 1M, Resistor_SMD:R_0402_1005Metric, F.Cu at (93.7, 91.7)
- added R38: 1M, Resistor_SMD:R_0402_1005Metric, F.Cu at (89.2, 95.6)
- added R39: 1Meg, Resistor_SMD:R_0402_1005Metric, F.Cu at (90.8, 91.7)
- added R4: 470, Resistor_SMD:R_0402_1005Metric, F.Cu at (18.3, 104.6)
- added R40: 1k, Resistor_SMD:R_0402_1005Metric, F.Cu at (87.9, 91.7)
- added R41: 499k, Resistor_SMD:R_0402_1005Metric, F.Cu at (90.8, 93.7)
- added R42: 1M, Resistor_SMD:R_0402_1005Metric, F.Cu at (15.2, 112.7)
- added R43: 1M, Resistor_SMD:R_0402_1005Metric, F.Cu at (21.0, 110.7)
- added R44: 1M, Resistor_SMD:R_0402_1005Metric, F.Cu at (16.5, 114.7)
- added R45: 1Meg, Resistor_SMD:R_0402_1005Metric, F.Cu at (18.1, 110.7)
- added R46: 1k, Resistor_SMD:R_0402_1005Metric, F.Cu at (15.2, 110.7)
- added R47: 499k, Resistor_SMD:R_0402_1005Metric, F.Cu at (18.1, 112.7)
- added R48: 1M, Resistor_SMD:R_0402_1005Metric, F.Cu at (70.5, 107.0)
- added R49: 1M, Resistor_SMD:R_0402_1005Metric, F.Cu at (76.3, 105.0)
- added R5: 470, Resistor_SMD:R_0402_1005Metric, F.Cu at (29.0, 103.8)
- added R50: 1M, Resistor_SMD:R_0402_1005Metric, F.Cu at (71.8, 109.0)
- added R51: 1Meg, Resistor_SMD:R_0402_1005Metric, F.Cu at (73.4, 105.0)
- added R52: 1k, Resistor_SMD:R_0402_1005Metric, F.Cu at (70.5, 105.0)
- added R53: 499k, Resistor_SMD:R_0402_1005Metric, F.Cu at (73.4, 107.0)
- added R6: 1M, Resistor_SMD:R_0402_1005Metric, F.Cu at (70.5, 93.7)
- added R7: 1M, Resistor_SMD:R_0402_1005Metric, F.Cu at (76.3, 91.7)
- added R8: 1M, Resistor_SMD:R_0402_1005Metric, F.Cu at (71.8, 95.6)
- added R9: 1Meg, Resistor_SMD:R_0402_1005Metric, F.Cu at (73.4, 91.7)
- added SW1: SW_User, Button_Switch_THT:SW_PUSH_6mm, F.Cu at (23.6, 79.3)
- added U1: STM32F072C8Tx, Package_QFP:LQFP-48_7x7mm_P0.5mm, F.Cu at (15.5, 93.5)
- added U10: LMP7715, Package_TO_SOT_SMD:SOT-23-5, F.Cu at (67.7, 111.6)
- added U2: MIC5205-3.3YM5, Package_TO_SOT_SMD:SOT-23-5, F.Cu at (18.0, 101.4)
- added U3: LMP7715, Package_TO_SOT_SMD:SOT-23-5, F.Cu at (67.7, 98.2)
- added U4: LMP7715, Package_TO_SOT_SMD:SOT-23-5, F.Cu at (47.4, 117.3)
- added U5: LMP7715, Package_TO_SOT_SMD:SOT-23-5, F.Cu at (29.9, 117.3)
- added U6: LMP7715, Package_TO_SOT_SMD:SOT-23-5, F.Cu at (67.7, 84.9)
- added U7: LMP7715, Package_TO_SOT_SMD:SOT-23-5, F.Cu at (85.2, 84.9)
- added U8: LMP7715, Package_TO_SOT_SMD:SOT-23-5, F.Cu at (85.2, 98.2)
- added U9: LMP7715, Package_TO_SOT_SMD:SOT-23-5, F.Cu at (12.4, 117.3)
Other:
- board outline added: 100 x 100 mm
- copper layers 0 -> 2
