File: hardware/microphone.kicad_sch (KiCad schematic)
At the start: 15 parts, among them U10 LMP7715

Commit message: Remove 4 of the 8 mounting holes
Parts:
- renumbered C58 to C30, C59 to C31, C60 to C32, C61 to C33, C62 to C34, C63 to C35, C64 to C36, MK8 to MK4, R48 to R24, R49 to R25, R50 to R26, R51 to R27, R52 to R28, R53 to R29, U10 to U6
Changed lines of the file:
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@@
   (symbol (lib_id "power:+3V3") (at 205.74 45.72 0)
     (in_bom yes) (on_board yes)
-    (property "Reference" "#PWR0127" (id 0) (at 205.74 49.53 0)
+    (property "Reference" "#PWR067" (id 0) (at 205.74 49.53 0)
       (effects (font (size 1.27 1.27)) hide)
     )
@@
   (symbol (lib_id "power:+3V3") (at 205.74 68.58 0)
     (in_bom yes) (on_board yes)
-    (property "Reference" "#PWR0129" (id 0) (at 205.74 72.39 0)
+    (property "Reference" "#PWR069" (id 0) (at 205.74 72.39 0)
       (effects (font (size 1.27 1.27)) hide)
     )
@@
   (symbol (lib_id "power:+3V3") (at 218.44 88.9 0)
     (in_bom yes) (on_board yes)
-    (property "Reference" "#PWR0131" (id 0) (at 218.44 92.71 0)
+    (property "Reference" "#PWR071" (id 0) (at 218.44 92.71 0)
       (effects (font (size 1.27 1.27)) hide)
     )
@@
   (symbol (lib_id "power:+3V3") (at 248.92 45.72 0)
     (in_bom yes) (on_board yes)
-    (property "Reference" "#PWR0135" (id 0) (at 248.92 49.53 0)
+    (property "Reference" "#PWR075" (id 0) (at 248.92 49.53 0)
       (effects (font (size 1.27 1.27)) hide)
     )
@@
   (symbol (lib_id "power:+3V3") (at 256.54 45.72 0)
     (in_bom yes) (on_board yes)
-    (property "Reference" "#PWR0138" (id 0) (at 256.54 49.53 0)
+    (property "Reference" "#PWR078" (id 0) (at 256.54 49.53 0)
       (effects (font (size 1.27 1.27)) hide)
     )
@@
   (symbol (lib_id "power:+3V3") (at 256.54 71.12 0)
     (in_bom yes) (on_board yes)
-    (property "Reference" "#PWR0140" (id 0) (at 256.54 74.93 0)
+    (property "Reference" "#PWR080" (id 0) (at 256.54 74.93 0)
       (effects (font (size 1.27 1.27)) hide)
     )
@@
   (symbol (lib_id "power:GND") (at 205.74 55.88 0)
     (in_bom yes) (on_board yes)
-    (property "Reference" "#PWR0128" (id 0) (at 205.74 62.23 0)
+    (property "Reference" "#PWR068" (id 0) (at 205.74 62.23 0)
       (effects (font (size 1.27 1.27)) hide)
     )
@@
   (symbol (lib_id "power:GND") (at 205.74 88.9 0)
     (in_bom yes) (on_board yes)
-    (property "Reference" "#PWR0130" (id 0) (at 205.74 95.25 0)
+    (property "Reference" "#PWR070" (id 0) (at 205.74 95.25 0)
       (effects (font (size 1.27 1.27)) hide)
     )
@@
   (symbol (lib_id "power:GND") (at 218.44 109.22 0)
     (in_bom yes) (on_board yes)
-    (property "Reference" "#PWR0132" (id 0) (at 218.44 115.57 0)
+    (property "Reference" "#PWR072" (id 0) (at 218.44 115.57 0)
       (effects (font (size 1.27 1.27)) hide)
     )
@@
   (symbol (lib_id "power:GND") (at 226.06 109.22 0)
     (in_bom yes) (on_board yes)
-    (property "Reference" "#PWR0133" (id 0) (at 226.06 115.57 0)
+    (property "Reference" "#PWR073" (id 0) (at 226.06 115.57 0)
       (effects (font (size 1.27 1.27)) hide)
     )
@@
   (symbol (lib_id "power:GND") (at 236.22 109.22 0)
     (in_bom yes) (on_board yes)
-    (property "Reference" "#PWR0134" (id 0) (at 236.22 115.57 0)
+    (property "Reference" "#PWR074" (id 0) (at 236.22 115.57 0)
       (effects (font (size 1.27 1.27)) hide)
     )
@@
   (symbol (lib_id "power:GND") (at 248.92 55.88 0)
     (in_bom yes) (on_board yes)
-    (property "Reference" "#PWR0136" (id 0) (at 248.92 62.23 0)
+    (property "Reference" "#PWR076" (id 0) (at 248.92 62.23 0)
       (effects (font (size 1.27 1.27)) hide)
     )
@@
   (symbol (lib_id "power:GND") (at 248.92 121.92 0)
     (in_bom yes) (on_board yes)
-    (property "Reference" "#PWR0137" (id 0) (at 248.92 128.27 0)
+    (property "Reference" "#PWR077" (id 0) (at 248.92 128.27 0)
       (effects (font (size 1.27 1.27)) hide)
     )
@@
   (symbol (lib_id "power:GND") (at 256.54 55.88 0)
     (in_bom yes) (on_board yes)
-    (property "Reference" "#PWR0139" (id 0) (at 256.54 62.23 0)
+    (property "Reference" "#PWR079" (id 0) (at 256.54 62.23 0)
       (effects (font (size 1.27 1.27)) hide)
     )
@@
   (symbol (lib_id "power:GND") (at 256.54 91.44 0)
     (in_bom yes) (on_board yes)
-    (property "Reference" "#PWR0141" (id 0) (at 256.54 97.79 0)
+    (property "Reference" "#PWR081" (id 0) (at 256.54 97.79 0)
       (effects (font (size 1.27 1.27)) hide)
     )
@@
   (symbol (lib_id "Device:R_Small") (at 218.44 93.98 0)
     (in_bom yes) (on_board yes)
-    (property "Reference" "R48" (id 0) (at 219.9387 92.8306 0)
+    (property "Reference" "R24" (id 0) (at 219.9387 92.8306 0)
       (effects (font (size 1.27 1.27)) (justify left))
     )
@@
   (symbol (lib_id "Device:R_Small") (at 218.44 104.14 0)
     (in_bom yes) (on_board yes)
-    (property "Reference" "R49" (id 0) (at 219.9387 102.9906 0)
+    (property "Reference" "R25" (id 0) (at 219.9387 102.9906 0)
       (effects (font (size 1.27 1.27)) (justify left))
     )
@@
   (symbol (lib_id "Device:R_Small") (at 231.14 99.06 90)
     (in_bom yes) (on_board yes)
-    (property "Reference" "R50" (id 0) (at 229.9906 97.5613 0)
+    (property "Reference" "R26" (id 0) (at 229.9906 97.5613 0)
       (effects (font (size 1.27 1.27)) (justify left))
     )
@@
   (symbol (lib_id "Device:R_Small") (at 236.22 88.9 0)
     (in_bom yes) (on_board yes)
-    (property "Reference" "R51" (id 0) (at 237.7187 87.7506 0)
+    (property "Reference" "R27" (id 0) (at 237.7187 87.7506 0)
       (effects (font (size 1.27 1.27)) (justify left))
     )
@@
   (symbol (lib_id "Device:R_Small") (at 248.92 109.22 180)
     (in_bom yes) (on_board yes)
-    (property "Reference" "R52" (id 0) (at 243.9732 109.22 90))
+    (property "Reference" "R28" (id 0) (at 243.9732 109.22 90))
     (property "Value" "1k" (id 1) (at 246.2784 109.22 90))
     (property "Footprint" "Resistor_SMD:R_0402_1005Metric" (id 2) (at 248.92 109.22 0)
@@
   (symbol (lib_id "Device:R_Small") (at 259.08 104.14 90)
     (in_bom yes) (on_board yes)
-    (property "Reference" "R53" (id 0) (at 259.08 99.1932 90))
+    (property "Reference" "R29" (id 0) (at 259.08 99.1932 90))
     (property "Value" "499k" (id 1) (at 259.08 101.4984 90))
     (property "Footprint" "Resistor_SMD:R_0402_1005Metric" (id 2) (at 259.08 104.14 0)
@@
   (symbol (lib_id "Device:C_Small") (at 205.74 50.8 0)
     (in_bom yes) (on_board yes)
-    (property "Reference" "C58" (id 0) (at 208.0642 49.6506 0)
+    (property "Reference" "C30" (id 0) (at 208.0642 49.6506 0)
       (effects (font (size 1.27 1.27)) (justify left))
     )
@@
   (symbol (lib_id "Device:C_Small") (at 220.98 78.74 90)
     (in_bom yes) (on_board yes)
-    (property "Reference" "C59" (id 0) (at 220.98 72.9677 90))
+    (property "Reference" "C31" (id 0) (at 220.98 72.9677 90))
     (property "Value" "1u" (id 1) (at 220.98 75.2602 90))
     (property "Footprint" "Capacitor_SMD:C_0402_1005Metric" (id 2) (at 220.98 78.74 0)
@@
   (symbol (lib_id "Device:C_Small") (at 226.06 104.14 0)
     (in_bom yes) (on_board yes)
-    (property "Reference" "C60" (id 0) (at 228.3842 102.9906 0)
+    (property "Reference" "C32" (id 0) (at 228.3842 102.9906 0)
       (effects (font (size 1.27 1.27)) (justify left))
     )
@@
   (symbol (lib_id "Device:C_Small") (at 236.22 104.14 0)
     (in_bom yes) (on_board yes)
-    (property "Reference" "C61" (id 0) (at 238.5442 102.9906 0)
+    (property "Reference" "C33" (id 0) (at 238.5442 102.9906 0)
       (effects (font (size 1.27 1.27)) (justify left))
     )
@@
   (symbol (lib_id "Device:C_Small") (at 248.92 50.8 0)
     (in_bom yes) (on_board yes)
-    (property "Reference" "C62" (id 0) (at 251.2442 49.6506 0)
+    (property "Reference" "C34" (id 0) (at 251.2442 49.6506 0)
       (effects (font (size 1.27 1.27)) (justify left))
     )
@@
   (symbol (lib_id "Device:C_Small") (at 248.92 116.84 0)
     (in_bom yes) (on_board yes)
-    (property "Reference" "C63" (id 0) (at 251.2442 115.6906 0)
+    (property "Reference" "C35" (id 0) (at 251.2442 115.6906 0)
       (effects (font (size 1.27 1.27)) (justify left))
     )
@@
   (symbol (lib_id "Device:C_Small") (at 256.54 50.8 0)
     (in_bom yes) (on_board yes)
-    (property "Reference" "C64" (id 0) (at 258.8642 49.6506 0)
+    (property "Reference" "C36" (id 0) (at 258.8642 49.6506 0)
       (effects (font (size 1.27 1.27)) (justify left))
     )
@@
   (symbol (lib_id "User:LMP7715") (at 259.08 81.28 0)
     (in_bom yes) (on_board yes)
-    (property "Reference" "U10" (id 0) (at 262.6361 77.5906 0)
+    (property "Reference" "U6" (id 0) (at 262.6361 77.5906 0)
       (effects (font (size 1.27 1.27)) (justify left))
     )
@@
   (symbol (lib_id "User:AP3722AT") (at 205.74 78.74 0)
     (in_bom yes) (on_board yes)
-    (property "Reference" "MK8" (id 0) (at 197.358 77.5906 0)
+    (property "Reference" "MK4" (id 0) (at 197.358 77.5906 0)
       (effects (font (size 1.27 1.27)) (justify right))
     )
